Commit message: Add files via upload

File: src/robot_description/urdf/robot.urdf.xacro (robot description, xacro)
@@ -49,5 +49,5 @@
         <parent link="base_link" />
         <child link="right_wheel_link" />
-        <origin xyz="0 0.09 0" rpy="${pi/2} 0 0" />
+        <origin xyz="0 0.09 0" rpy="1.5708 0 0" />
         <axis xyz="0 0 1" />
     </joint>
@@ -66,5 +66,5 @@
         <parent link="base_link" />
         <child link="left_wheel_link" />
-        <origin xyz="0 -0.09 0" rpy=" ${pi/2} 0 0" />
+        <origin xyz="0 -0.09 0" rpy=" 1.5708 0 0" />
         <axis xyz="0 0 1" />
     </joint>
